File: phy_adm.sch (KiCad schematic (older format))
At the start: 28 parts

Commit message: sch: Misc fixes
Connections:
- net GND: now also U?.3 (GND)
Changed lines of the file:
@@
 $Descr A4 11693 8268
 encoding utf-8
-Sheet 4 9
+Sheet 4 10
 Title "PHY control plane"
 Date "2019-03-19"
@@
 Wire Wire Line
 	5100 1400 5200 1400
-Text Label 5150 1700 0    50   ~ 0
+Text Label 5600 1700 2    50   ~ 0
 REF_CLK_P
-Text Label 5150 1800 0    50   ~ 0
+Text Label 5600 1800 2    50   ~ 0
 REF_CLK_N
 Wire Wire Line
@@
 Text Label 2200 3100 0    50   ~ 0
 LED_P3_0
+$Comp
+L power:GND #PWR?
+U 1 1 5D465DF9
+P 4500 5750
+F 0 "#PWR?" H 4500 5500 50  0001 C CNN
+F 1 "GND" H 4505 5577 50  0000 C CNN
+F 2 "" H 4500 5750 50  0001 C CNN
+F 3 "" H 4500 5750 50  0001 C CNN
+	1    4500 5750
+	1    0    0    -1
+$EndComp
+Wire Wire Line
+	4600 5500 4500 5500
+Wire Wire Line
+	4500 5500 4500 5750
 $EndSCHEMATC
