File: usb-uart.sch (KiCad schematic (older format))
At the start: 11 parts

Commit message: sch: Misc fixes
Parts:
- C?: value C -> 100n
Changed lines of the file:
@@
 $Descr A4 11693 8268
 encoding utf-8
-Sheet 7 9
+Sheet 7 10
 Title "USB to UART conversion"
 Date "2019-03-19"
@@
 P 7250 3200
 F 0 "C?" V 6998 3200 50  0000 C CNN
-F 1 "C" V 7089 3200 50  0000 C CNN
+F 1 "100n" V 7089 3200 50  0000 C CNN
 F 2 "" H 7288 3050 50  0001 C CNN
 F 3 "~" H 7250 3200 50  0001 C CNN
