File: pimouss-motherboard.sch (KiCad schematic (older format))
At the start: 2 parts

Commit message: sch: Annotate & associate symbols with footprints
Parts:
- removed DS?: DummySupply, symbol pimouss-motherboard:DummySupply
- R1: renamed from R?; footprint (none) -> Resistor_SMD:R_0603_1608Metric
Changed lines of the file:
@@
 LED_P3_0
 $Comp
-L power:GND #PWR?
+L power:GND #PWR01
 U 1 1 5E474FB1
 P 4000 6700
-F 0 "#PWR?" H 4000 6450 50  0001 C CNN
+F 0 "#PWR01" H 4000 6450 50  0001 C CNN
 F 1 "GND" H 4005 6527 50  0000 C CNN
 F 2 "" H 4000 6700 50  0001 C CNN
@@
 $EndComp
 $Comp
-L power:Earth #PWR?
+L power:Earth #PWR02
 U 1 1 5E475AA8
 P 4400 6700
-F 0 "#PWR?" H 4400 6450 50  0001 C CNN
+F 0 "#PWR02" H 4400 6450 50  0001 C CNN
 F 1 "Earth" H 4400 6550 50  0001 C CNN
 F 2 "" H 4400 6700 50  0001 C CNN
@@
 $EndComp
 $Comp
-L pimouss-motherboard:DummySupply DS?
+L pimouss-motherboard:DummySupply #DS01
 U 1 1 5E47640A
 P 4400 6600
-F 0 "DS?" H 4400 6600 50  0001 C CNN
+F 0 "#DS01" H 4400 6600 50  0001 C CNN
 F 1 "DummySupply" H 4400 6600 50  0001 C CNN
 F 2 "" H 4400 6600 50  0001 C CNN
@@
 $EndComp
 $Comp
-L Device:R_Small R?
+L Device:R_Small R1
 U 1 1 5E476DB3
 P 4200 6600
-F 0 "R?" V 4004 6600 50  0000 C CNN
+F 0 "R1" V 4004 6600 50  0000 C CNN
 F 1 "1M" V 4095 6600 50  0000 C CNN
-F 2 "" H 4200 6600 50  0001 C CNN
+F 2 "Resistor_SMD:R_0603_1608Metric" H 4200 6600 50  0001 C CNN
 F 3 "~" H 4200 6600 50  0001 C CNN
 	1    4200 6600
