File: pcie_mpcie.sch (KiCad schematic (older format))
At the start: 9 parts

Commit message: sch: Replace regular symbols with small variant
Done for most capacitors and resistors
Parts:
- removed C? (x2): 100n, symbol Device:C
- removed R? (x3): 270, symbol Device:R
- added C? (x2): 100n, symbol Device:C_Small
- added R? (x3): 270, symbol Device:R_Small
Other:
- moved on the sheet: D?
Changed lines of the file:
@@
 	4800 3600 3250 3600
 Wire Wire Line
-	4000 3900 3250 3900
-Wire Wire Line
-	4000 4000 3250 4000
+	4050 3900 3250 3900
+Wire Wire Line
+	4050 4000 3250 4000
 Text Label 3300 4600 0    50   ~ 0
 PCIE_X1_CLK_P
@@
 Text Label 6450 4100 0    50   ~ 0
 nRST
-$Comp
-L Device:C C?
-U 1 1 5D4896AE
-P 4150 3900
-AR Path="/5C91A44F/5D4896AE" Ref="C?"  Part="1"
-AR Path="/5C91A44F/5D489567/5D4896AE" Ref="C?"  Part="1"
-AR Path="/5C91A44F/5D9DAD5B/5D4896AE" Ref="C?"  Part="1"
-AR Path="/5C91A44F/5D9F9D59/5D4896AE" Ref="C?"  Part="1"
-F 0 "C?" V 4100 3850 50  0000 R BNN
-F 1 "100n" V 4100 3950 50  0000 L BNN
-F 2 "" H 4188 3750 50  0001 C CNN
-F 3 "~" H 4150 3900 50  0001 C CNN
-	1    4150 3900
-	0    -1   1    0
-$EndComp
-$Comp
-L Device:C C?
-U 1 1 5D4896B5
-P 4150 4000
-AR Path="/5C91A44F/5D4896B5" Ref="C?"  Part="1"
-AR Path="/5C91A44F/5D489567/5D4896B5" Ref="C?"  Part="1"
-AR Path="/5C91A44F/5D9DAD5B/5D4896B5" Ref="C?"  Part="1"
-AR Path="/5C91A44F/5D9F9D59/5D4896B5" Ref="C?"  Part="1"
-F 0 "C?" V 4200 3950 50  0000 R TNN
-F 1 "100n" V 4200 4050 50  0000 L TNN
-F 2 "" H 4188 3850 50  0001 C CNN
-F 3 "~" H 4150 4000 50  0001 C CNN
-	1    4150 4000
-	0    -1   1    0
-$EndComp
 Text Label 4650 3900 2    50   ~ 0
 X1_R_P
@@
 	4800 4700 3250 4700
 Wire Wire Line
-	4800 3900 4300 3900
-Wire Wire Line
-	4800 4000 4300 4000
+	4800 3900 4250 3900
+Wire Wire Line
+	4800 4000 4250 4000
 $Comp
 L mpcie:MPCIE-Socket U?
@@
 L Device:LED D?
 U 1 1 5D48971E
-P 7000 2250
+P 7000 2350
 AR Path="/5C91A44F/5D48971E" Ref="D?"  Part="1"
 AR Path="/5C91A44F/5D489567/5D48971E" Ref="D?"  Part="1"
 AR Path="/5C91A44F/5D9DAD5B/5D48971E" Ref="D?"  Part="1"
 AR Path="/5C91A44F/5D9F9D59/5D48971E" Ref="D?"  Part="1"
-F 0 "D?" V 7038 2132 50  0000 R CNN
-F 1 "G" V 6947 2132 50  0000 R CNN
-F 2 "" H 7000 2250 50  0001 C CNN
-F 3 "~" H 7000 2250 50  0001 C CNN
-	1    7000 2250
+F 0 "D?" V 7038 2232 50  0000 R CNN
+F 1 "G" V 6947 2232 50  0000 R CNN
+F 2 "" H 7000 2350 50  0001 C CNN
+F 3 "~" H 7000 2350 50  0001 C CNN
+	1    7000 2350
 	0    -1   -1   0
 $EndComp
@@
 L Device:LED D?
 U 1 1 5D489725
-P 7300 2250
+P 7300 2350
 AR Path="/5C91A44F/5D489725" Ref="D?"  Part="1"
 AR Path="/5C91A44F/5D489567/5D489725" Ref="D?"  Part="1"
 AR Path="/5C91A44F/5D9DAD5B/5D489725" Ref="D?"  Part="1"
 AR Path="/5C91A44F/5D9F9D59/5D489725" Ref="D?"  Part="1"
-F 0 "D?" V 7338 2132 50  0000 R CNN
-F 1 "R" V 7247 2132 50  0000 R CNN
-F 2 "" H 7300 2250 50  0001 C CNN
-F 3 "~" H 7300 2250 50  0001 C CNN
-	1    7300 2250
+F 0 "D?" V 7338 2232 50  0000 R CNN
+F 1 "R" V 7247 2232 50  0000 R CNN
+F 2 "" H 7300 2350 50  0001 C CNN
+F 3 "~" H 7300 2350 50  0001 C CNN
+	1    7300 2350
 	0    -1   -1   0
 $EndComp
@@
 L Device:LED D?
 U 1 1 5D48972C
-P 7600 2250
+P 7600 2350
 AR Path="/5C91A44F/5D48972C" Ref="D?"  Part="1"
 AR Path="/5C91A44F/5D489567/5D48972C" Ref="D?"  Part="1"
 AR Path="/5C91A44F/5D9DAD5B/5D48972C" Ref="D?"  Part="1"
 AR Path="/5C91A44F/5D9F9D59/5D48972C" Ref="D?"  Part="1"
-F 0 "D?" V 7638 2132 50  0000 R CNN
-F 1 "Y" V 7547 2132 50  0000 R CNN
-F 2 "" H 7600 2250 50  0001 C CNN
-F 3 "~" H 7600 2250 50  0001 C CNN
-	1    7600 2250
+F 0 "D?" V 7638 2232 50  0000 R CNN
+F 1 "Y" V 7547 2232 50  0000 R CNN
+F 2 "" H 7600 2350 50  0001 C CNN
+F 3 "~" H 7600 2350 50  0001 C CNN
+	1    7600 2350
 	0    -1   -1   0
 $EndComp
-$Comp
-L Device:R R?
-U 1 1 5D489733
-P 7000 2650
-AR Path="/5C91A44F/5D489733" Ref="R?"  Part="1"
-AR Path="/5C91A44F/5D489567/5D489733" Ref="R?"  Part="1"
-AR Path="/5C91A44F/5D9DAD5B/5D489733" Ref="R?"  Part="1"
-AR Path="/5C91A44F/5D9F9D59/5D489733" Ref="R?"  Part="1"
-F 0 "R?" H 7070 2696 50  0000 L CNN
-F 1 "270" H 7070 2605 50  0000 L CNN
-F 2 "" V 6930 2650 50  0001 C CNN
-F 3 "~" H 7000 2650 50  0001 C CNN
-	1    7000 2650
-	1    0    0    -1
-$EndComp
 Wire Wire Line
 	6100 2900 7000 2900
@@
 	6100 3100 7600 3100
 Wire Wire Line
-	7000 2400 7000 2500
-Wire Wire Line
-	7300 2400 7300 2500
-Wire Wire Line
-	7600 2400 7600 2500
-Wire Wire Line
-	7000 2100 7000 2000
-Wire Wire Line
-	7600 2000 7600 2100
-Wire Wire Line
-	7300 2100 7300 2000
-Wire Wire Line
-	7000 2000 7300 2000
-Connection ~ 7300 2000
-Wire Wire Line
-	7300 2000 7600 2000
+	7000 2500 7000 2600
+Wire Wire Line
+	7300 2500 7300 2600
+Wire Wire Line
+	7600 2500 7600 2600
+Wire Wire Line
+	7000 2200 7000 2100
+Wire Wire Line
+	7600 2100 7600 2200
+Wire Wire Line
+	7300 2200 7300 2100
+Wire Wire Line
+	7000 2100 7300 2100
+Connection ~ 7300 2100
+Wire Wire Line
+	7300 2100 7600 2100
 $Comp
 L power:+3V3 #PWR?
 U 1 1 5D489749
-P 7300 1900
+P 7300 2000
 AR Path="/5C91A44F/5D489749" Ref="#PWR?"  Part="1"
 AR Path="/5C91A44F/5D489567/5D489749" Ref="#PWR?"  Part="1"
 AR Path="/5C91A44F/5D9DAD5B/5D489749" Ref="#PWR?"  Part="1"
 AR Path="/5C91A44F/5D9F9D59/5D489749" Ref="#PWR?"  Part="1"
-F 0 "#PWR?" H 7300 1750 50  0001 C CNN
-F 1 "+3V3" H 7315 2073 50  0000 C CNN
-F 2 "" H 7300 1900 50  0001 C CNN
-F 3 "" H 7300 1900 50  0001 C CNN
-	1    7300 1900
-	1    0    0    -1
-$EndComp
-Wire Wire Line
-	7300 1900 7300 2000
-$Comp
-L Device:R R?
-U 1 1 5D489750
-P 7300 2650
-AR Path="/5C91A44F/5D489750" Ref="R?"  Part="1"
-AR Path="/5C91A44F/5D489567/5D489750" Ref="R?"  Part="1"
-AR Path="/5C91A44F/5D9DAD5B/5D489750" Ref="R?"  Part="1"
-AR Path="/5C91A44F/5D9F9D59/5D489750" Ref="R?"  Part="1"
-F 0 "R?" H 7370 2696 50  0000 L CNN
-F 1 "270" H 7370 2605 50  0000 L CNN
-F 2 "" V 7230 2650 50  0001 C CNN
-F 3 "~" H 7300 2650 50  0001 C CNN
-	1    7300 2650
-	1    0    0    -1
-$EndComp
-$Comp
-L Device:R R?
-U 1 1 5D489757
-P 7600 2650
-AR Path="/5C91A44F/5D489757" Ref="R?"  Part="1"
-AR Path="/5C91A44F/5D489567/5D489757" Ref="R?"  Part="1"
-AR Path="/5C91A44F/5D9DAD5B/5D489757" Ref="R?"  Part="1"
-AR Path="/5C91A44F/5D9F9D59/5D489757" Ref="R?"  Part="1"
-F 0 "R?" H 7670 2696 50  0000 L CNN
-F 1 "270" H 7670 2605 50  0000 L CNN
-F 2 "" V 7530 2650 50  0001 C CNN
-F 3 "~" H 7600 2650 50  0001 C CNN
-	1    7600 2650
-	1    0    0    -1
-$EndComp
+F 0 "#PWR?" H 7300 1850 50  0001 C CNN
+F 1 "+3V3" H 7315 2173 50  0000 C CNN
+F 2 "" H 7300 2000 50  0001 C CNN
+F 3 "" H 7300 2000 50  0001 C CNN
+	1    7300 2000
+	1    0    0    -1
+$EndComp
+Wire Wire Line
+	7300 2000 7300 2100
 $Comp
 L pimouss-motherboard:+1V5_PCI #PWR?
@@
 Text Label 3300 3500 0    50   ~ 0
 PCIE_X1_TX_P
+$Comp
+L Device:R_Small R?
+U 1 1 5D47B705
+P 7600 2700
+F 0 "R?" H 7659 2746 50  0000 L CNN
+F 1 "270" H 7659 2655 50  0000 L CNN
+F 2 "" H 7600 2700 50  0001 C CNN
+F 3 "~" H 7600 2700 50  0001 C CNN
+	1    7600 2700
+	1    0    0    -1
+$EndComp
+$Comp
+L Device:R_Small R?
+U 1 1 5D47DB0E
+P 7000 2700
+F 0 "R?" H 7059 2746 50  0000 L CNN
+F 1 "270" H 7059 2655 50  0000 L CNN
+F 2 "" H 7000 2700 50  0001 C CNN
+F 3 "~" H 7000 2700 50  0001 C CNN
+	1    7000 2700
+	1    0    0    -1
+$EndComp
+$Comp
+L Device:R_Small R?
+U 1 1 5D47E3D4
+P 7300 2700
+F 0 "R?" H 7359 2746 50  0000 L CNN
+F 1 "270" H 7359 2655 50  0000 L CNN
+F 2 "" H 7300 2700 50  0001 C CNN
+F 3 "~" H 7300 2700 50  0001 C CNN
+	1    7300 2700
+	1    0    0    -1
+$EndComp
+$Comp
+L Device:C_Small C?
+U 1 1 5D48454A
+P 4150 4000
+F 0 "C?" V 4250 3900 50  0000 C CNN
+F 1 "100n" V 4250 4150 50  0000 C CNN
+F 2 "" H 4150 4000 50  0001 C CNN
+F 3 "~" H 4150 4000 50  0001 C CNN
+	1    4150 4000
+	0    -1   1    0
+$EndComp
+$Comp
+L Device:C_Small C?
+U 1 1 5D484550
+P 4150 3900
+F 0 "C?" V 4050 3800 50  0000 C CNN
+F 1 "100n" V 4050 4050 50  0000 C CNN
+F 2 "" H 4150 3900 50  0001 C CNN
+F 3 "~" H 4150 3900 50  0001 C CNN
+	1    4150 3900
+	0    -1   1    0
+$EndComp
 $EndSCHEMATC

Commit message: lib: Move mPCIe socket to local lib
Parts:
- removed U?: MPCIE-Socket, symbol mpcie:MPCIE-Socket
- added U?: MPCIE-Socket, pimouss-motherboard:mpcie-socket, symbol pimouss-motherboard:MPCIE-Socket
Changed lines of the file:
@@
 Wire Wire Line
 	4800 4000 4250 4000
-$Comp
-L mpcie:MPCIE-Socket U?
-U 1 1 5D4896C2
-P 5450 3750
-AR Path="/5C91A44F/5D4896C2" Ref="U?"  Part="1"
-AR Path="/5C91A44F/5D489567/5D4896C2" Ref="U?"  Part="1"
-AR Path="/5C91A44F/5D9DAD5B/5D4896C2" Ref="U?"  Part="1"
-AR Path="/5C91A44F/5D9F9D59/5D4896C2" Ref="U?"  Part="1"
-F 0 "U?" H 5450 5187 60  0000 C CNN
-F 1 "MPCIE-Socket" H 5450 5081 60  0000 C CNN
-F 2 "" H 5550 2750 60  0000 C CNN
-F 3 "" H 5550 2750 60  0000 C CNN
-	1    5450 3750
-	1    0    0    -1
-$EndComp
 Wire Wire Line
 	4800 3000 4700 3000
@@
 	0    -1   1    0
 $EndComp
+$Comp
+L pimouss-motherboard:MPCIE-Socket U?
+U 1 1 5E649649
+P 5450 3750
+F 0 "U?" H 5450 5293 60  0000 C CNN
+F 1 "MPCIE-Socket" H 5450 5187 60  0000 C CNN
+F 2 "pimouss-motherboard:mpcie-socket" H 5450 5081 60  0000 C CNN
+F 3 "" H 5550 2750 60  0000 C CNN
+	1    5450 3750
+	1    0    0    -1
+$EndComp
 $EndSCHEMATC

Commit message: sch: Annotate & associate symbols with footprints
Parts:
- C30, C31: renamed from C?; footprint (none) -> Capacitor_SMD:C_0402_1005Metric
- D1, D2, D3: renamed from D?; footprint (none) -> Diode_SMD:D_0603_1608Metric
- R38, R39, R40: renamed from R?; footprint (none) -> Resistor_SMD:R_0603_1608Metric
- gave numbers to parts that had none: 1
Changed lines of the file:
@@
 P 4700 5300
 AR Path="/5C91A44F/5D4896F1" Ref="#PWR?"  Part="1"
-AR Path="/5C91A44F/5D489567/5D4896F1" Ref="#PWR?"  Part="1"
+AR Path="/5C91A44F/5D489567/5D4896F1" Ref="#PWR065"  Part="1"
 AR Path="/5C91A44F/5D9DAD5B/5D4896F1" Ref="#PWR?"  Part="1"
-AR Path="/5C91A44F/5D9F9D59/5D4896F1" Ref="#PWR?"  Part="1"
-F 0 "#PWR?" H 4700 5050 50  0001 C CNN
+AR Path="/5C91A44F/5D9F9D59/5D4896F1" Ref="#PWR073"  Part="1"
+F 0 "#PWR073" H 4700 5050 50  0001 C CNN
 F 1 "GND" H 4705 5127 50  0000 C CNN
 F 2 "" H 4700 5300 50  0001 C CNN
@@
 P 6200 5300
 AR Path="/5C91A44F/5D4896F7" Ref="#PWR?"  Part="1"
-AR Path="/5C91A44F/5D489567/5D4896F7" Ref="#PWR?"  Part="1"
+AR Path="/5C91A44F/5D489567/5D4896F7" Ref="#PWR066"  Part="1"
 AR Path="/5C91A44F/5D9DAD5B/5D4896F7" Ref="#PWR?"  Part="1"
-AR Path="/5C91A44F/5D9F9D59/5D4896F7" Ref="#PWR?"  Part="1"
-F 0 "#PWR?" H 6200 5050 50  0001 C CNN
+AR Path="/5C91A44F/5D9F9D59/5D4896F7" Ref="#PWR074"  Part="1"
+F 0 "#PWR074" H 6200 5050 50  0001 C CNN
 F 1 "GND" H 6205 5127 50  0000 C CNN
 F 2 "" H 6200 5300 50  0001 C CNN
@@
 P 7000 2350
 AR Path="/5C91A44F/5D48971E" Ref="D?"  Part="1"
-AR Path="/5C91A44F/5D489567/5D48971E" Ref="D?"  Part="1"
+AR Path="/5C91A44F/5D489567/5D48971E" Ref="D1"  Part="1"
 AR Path="/5C91A44F/5D9DAD5B/5D48971E" Ref="D?"  Part="1"
-AR Path="/5C91A44F/5D9F9D59/5D48971E" Ref="D?"  Part="1"
-F 0 "D?" V 7038 2232 50  0000 R CNN
+AR Path="/5C91A44F/5D9F9D59/5D48971E" Ref="D4"  Part="1"
+F 0 "D1" V 7038 2232 50  0000 R CNN
 F 1 "G" V 6947 2232 50  0000 R CNN
-F 2 "" H 7000 2350 50  0001 C CNN
+F 2 "Diode_SMD:D_0603_1608Metric" H 7000 2350 50  0001 C CNN
 F 3 "~" H 7000 2350 50  0001 C CNN
 	1    7000 2350
@@
 P 7300 2350
 AR Path="/5C91A44F/5D489725" Ref="D?"  Part="1"
-AR Path="/5C91A44F/5D489567/5D489725" Ref="D?"  Part="1"
+AR Path="/5C91A44F/5D489567/5D489725" Ref="D2"  Part="1"
 AR Path="/5C91A44F/5D9DAD5B/5D489725" Ref="D?"  Part="1"
-AR Path="/5C91A44F/5D9F9D59/5D489725" Ref="D?"  Part="1"
-F 0 "D?" V 7338 2232 50  0000 R CNN
+AR Path="/5C91A44F/5D9F9D59/5D489725" Ref="D5"  Part="1"
+F 0 "D2" V 7338 2232 50  0000 R CNN
 F 1 "R" V 7247 2232 50  0000 R CNN
-F 2 "" H 7300 2350 50  0001 C CNN
+F 2 "Diode_SMD:D_0603_1608Metric" H 7300 2350 50  0001 C CNN
 F 3 "~" H 7300 2350 50  0001 C CNN
 	1    7300 2350
@@
 P 7600 2350
 AR Path="/5C91A44F/5D48972C" Ref="D?"  Part="1"
-AR Path="/5C91A44F/5D489567/5D48972C" Ref="D?"  Part="1"
+AR Path="/5C91A44F/5D489567/5D48972C" Ref="D3"  Part="1"
 AR Path="/5C91A44F/5D9DAD5B/5D48972C" Ref="D?"  Part="1"
-AR Path="/5C91A44F/5D9F9D59/5D48972C" Ref="D?"  Part="1"
-F 0 "D?" V 7638 2232 50  0000 R CNN
+AR Path="/5C91A44F/5D9F9D59/5D48972C" Ref="D6"  Part="1"
+F 0 "D3" V 7638 2232 50  0000 R CNN
 F 1 "Y" V 7547 2232 50  0000 R CNN
-F 2 "" H 7600 2350 50  0001 C CNN
+F 2 "Diode_SMD:D_0603_1608Metric" H 7600 2350 50  0001 C CNN
 F 3 "~" H 7600 2350 50  0001 C CNN
 	1    7600 2350
@@
 P 7300 2000
 AR Path="/5C91A44F/5D489749" Ref="#PWR?"  Part="1"
-AR Path="/5C91A44F/5D489567/5D489749" Ref="#PWR?"  Part="1"
+AR Path="/5C91A44F/5D489567/5D489749" Ref="#PWR071"  Part="1"
 AR Path="/5C91A44F/5D9DAD5B/5D489749" Ref="#PWR?"  Part="1"
-AR Path="/5C91A44F/5D9F9D59/5D489749" Ref="#PWR?"  Part="1"
-F 0 "#PWR?" H 7300 1850 50  0001 C CNN
+AR Path="/5C91A44F/5D9F9D59/5D489749" Ref="#PWR079"  Part="1"
+F 0 "#PWR079" H 7300 1850 50  0001 C CNN
 F 1 "+3V3" H 7315 2173 50  0000 C CNN
 F 2 "" H 7300 2000 50  0001 C CNN
@@
 P 6700 2500
 AR Path="/5C91A44F/5D48975F" Ref="#PWR?"  Part="1"
-AR Path="/5C91A44F/5D489567/5D48975F" Ref="#PWR?"  Part="1"
+AR Path="/5C91A44F/5D489567/5D48975F" Ref="#PWR069"  Part="1"
 AR Path="/5C91A44F/5D9DAD5B/5D48975F" Ref="#PWR?"  Part="1"
-AR Path="/5C91A44F/5D9F9D59/5D48975F" Ref="#PWR?"  Part="1"
-F 0 "#PWR?" H 6700 2350 50  0001 C CNN
+AR Path="/5C91A44F/5D9F9D59/5D48975F" Ref="#PWR077"  Part="1"
+F 0 "#PWR077" H 6700 2350 50  0001 C CNN
 F 1 "+1V5_PCI" H 6715 2673 50  0000 C CNN
 F 2 "" H 6700 2500 50  0001 C CNN
@@
 P 6300 2500
 AR Path="/5C91A44F/5D489765" Ref="#PWR?"  Part="1"
-AR Path="/5C91A44F/5D489567/5D489765" Ref="#PWR?"  Part="1"
+AR Path="/5C91A44F/5D489567/5D489765" Ref="#PWR067"  Part="1"
 AR Path="/5C91A44F/5D9DAD5B/5D489765" Ref="#PWR?"  Part="1"
-AR Path="/5C91A44F/5D9F9D59/5D489765" Ref="#PWR?"  Part="1"
-F 0 "#PWR?" H 6300 2350 50  0001 C CNN
+AR Path="/5C91A44F/5D9F9D59/5D489765" Ref="#PWR075"  Part="1"
+F 0 "#PWR075" H 6300 2350 50  0001 C CNN
 F 1 "+3V3_PCI" H 6315 2673 50  0000 C CNN
 F 2 "" H 6300 2500 50  0001 C CNN
@@
 P 4600 2500
 AR Path="/5C91A44F/5D48976B" Ref="#PWR?"  Part="1"
-AR Path="/5C91A44F/5D489567/5D48976B" Ref="#PWR?"  Part="1"
+AR Path="/5C91A44F/5D489567/5D48976B" Ref="#PWR064"  Part="1"
 AR Path="/5C91A44F/5D9DAD5B/5D48976B" Ref="#PWR?"  Part="1"
-AR Path="/5C91A44F/5D9F9D59/5D48976B" Ref="#PWR?"  Part="1"
-F 0 "#PWR?" H 4600 2350 50  0001 C CNN
+AR Path="/5C91A44F/5D9F9D59/5D48976B" Ref="#PWR072"  Part="1"
+F 0 "#PWR072" H 4600 2350 50  0001 C CNN
 F 1 "+3V3_PCI" H 4615 2673 50  0000 C CNN
 F 2 "" H 4600 2500 50  0001 C CNN
@@
 P 6400 4900
 AR Path="/5C91A44F/5D489771" Ref="#PWR?"  Part="1"
-AR Path="/5C91A44F/5D489567/5D489771" Ref="#PWR?"  Part="1"
+AR Path="/5C91A44F/5D489567/5D489771" Ref="#PWR068"  Part="1"
 AR Path="/5C91A44F/5D9DAD5B/5D489771" Ref="#PWR?"  Part="1"
-AR Path="/5C91A44F/5D9F9D59/5D489771" Ref="#PWR?"  Part="1"
-F 0 "#PWR?" H 6400 4750 50  0001 C CNN
+AR Path="/5C91A44F/5D9F9D59/5D489771" Ref="#PWR076"  Part="1"
+F 0 "#PWR076" H 6400 4750 50  0001 C CNN
 F 1 "+1V5_PCI" H 6415 5073 50  0000 C CNN
 F 2 "" H 6400 4900 50  0001 C CNN
@@
 P 6800 4900
 AR Path="/5C91A44F/5D489777" Ref="#PWR?"  Part="1"
-AR Path="/5C91A44F/5D489567/5D489777" Ref="#PWR?"  Part="1"
+AR Path="/5C91A44F/5D489567/5D489777" Ref="#PWR070"  Part="1"
 AR Path="/5C91A44F/5D9DAD5B/5D489777" Ref="#PWR?"  Part="1"
-AR Path="/5C91A44F/5D9F9D59/5D489777" Ref="#PWR?"  Part="1"
-F 0 "#PWR?" H 6800 4750 50  0001 C CNN
+AR Path="/5C91A44F/5D9F9D59/5D489777" Ref="#PWR078"  Part="1"
+F 0 "#PWR078" H 6800 4750 50  0001 C CNN
 F 1 "+3V3_PCI" H 6815 5073 50  0000 C CNN
 F 2 "" H 6800 4900 50  0001 C CNN
@@
 PCIE_X1_TX_P
 $Comp
-L Device:R_Small R?
+L Device:R_Small R40
 U 1 1 5D47B705
 P 7600 2700
-F 0 "R?" H 7659 2746 50  0000 L CNN
+AR Path="/5C91A44F/5D489567/5D47B705" Ref="R40"  Part="1"
+AR Path="/5C91A44F/5D9F9D59/5D47B705" Ref="R43"  Part="1"
+F 0 "R40" H 7659 2746 50  0000 L CNN
 F 1 "270" H 7659 2655 50  0000 L CNN
-F 2 "" H 7600 2700 50  0001 C CNN
+F 2 "Resistor_SMD:R_0603_1608Metric" H 7600 2700 50  0001 C CNN
 F 3 "~" H 7600 2700 50  0001 C CNN
 	1    7600 2700
@@
 $EndComp
 $Comp
-L Device:R_Small R?
+L Device:R_Small R38
 U 1 1 5D47DB0E
 P 7000 2700
-F 0 "R?" H 7059 2746 50  0000 L CNN
+AR Path="/5C91A44F/5D489567/5D47DB0E" Ref="R38"  Part="1"
+AR Path="/5C91A44F/5D9F9D59/5D47DB0E" Ref="R41"  Part="1"
+F 0 "R38" H 7059 2746 50  0000 L CNN
 F 1 "270" H 7059 2655 50  0000 L CNN
-F 2 "" H 7000 2700 50  0001 C CNN
+F 2 "Resistor_SMD:R_0603_1608Metric" H 7000 2700 50  0001 C CNN
 F 3 "~" H 7000 2700 50  0001 C CNN
 	1    7000 2700
@@
 $EndComp
 $Comp
-L Device:R_Small R?
+L Device:R_Small R39
 U 1 1 5D47E3D4
 P 7300 2700
-F 0 "R?" H 7359 2746 50  0000 L CNN
+AR Path="/5C91A44F/5D489567/5D47E3D4" Ref="R39"  Part="1"
+AR Path="/5C91A44F/5D9F9D59/5D47E3D4" Ref="R42"  Part="1"
+F 0 "R39" H 7359 2746 50  0000 L CNN
 F 1 "270" H 7359 2655 50  0000 L CNN
-F 2 "" H 7300 2700 50  0001 C CNN
+F 2 "Resistor_SMD:R_0603_1608Metric" H 7300 2700 50  0001 C CNN
 F 3 "~" H 7300 2700 50  0001 C CNN
 	1    7300 2700
@@
 $EndComp
 $Comp
-L Device:C_Small C?
+L Device:C_Small C31
 U 1 1 5D48454A
 P 4150 4000
-F 0 "C?" V 4250 3900 50  0000 C CNN
+AR Path="/5C91A44F/5D489567/5D48454A" Ref="C31"  Part="1"
+AR Path="/5C91A44F/5D9F9D59/5D48454A" Ref="C33"  Part="1"
+F 0 "C31" V 4250 3900 50  0000 C CNN
 F 1 "100n" V 4250 4150 50  0000 C CNN
-F 2 "" H 4150 4000 50  0001 C CNN
+F 2 "Capacitor_SMD:C_0402_1005Metric" H 4150 4000 50  0001 C CNN
 F 3 "~" H 4150 4000 50  0001 C CNN
 	1    4150 4000
@@
 $EndComp
 $Comp
-L Device:C_Small C?
+L Device:C_Small C30
 U 1 1 5D484550
 P 4150 3900
-F 0 "C?" V 4050 3800 50  0000 C CNN
+AR Path="/5C91A44F/5D489567/5D484550" Ref="C30"  Part="1"
+AR Path="/5C91A44F/5D9F9D59/5D484550" Ref="C32"  Part="1"
+F 0 "C30" V 4050 3800 50  0000 C CNN
 F 1 "100n" V 4050 4050 50  0000 C CNN
-F 2 "" H 4150 3900 50  0001 C CNN
+F 2 "Capacitor_SMD:C_0402_1005Metric" H 4150 3900 50  0001 C CNN
 F 3 "~" H 4150 3900 50  0001 C CNN
 	1    4150 3900
@@
 $EndComp
 $Comp
-L pimouss-motherboard:MPCIE-Socket U?
+L pimouss-motherboard:MPCIE-Socket U4
 U 1 1 5E649649
 P 5450 3750
-F 0 "U?" H 5450 5293 60  0000 C CNN
+AR Path="/5C91A44F/5D489567/5E649649" Ref="U4"  Part="1"
+AR Path="/5C91A44F/5D9F9D59/5E649649" Ref="U5"  Part="1"
+F 0 "U4" H 5450 5293 60  0000 C CNN
 F 1 "MPCIE-Socket" H 5450 5187 60  0000 C CNN
 F 2 "pimouss-motherboard:mpcie-socket" H 5450 5081 60  0000 C CNN

Commit message: lib, sch: Fix connectors refdes letter
Parts:
- renumbered U4 to P3
Changed lines of the file:
@@
 $EndComp
 $Comp
-L pimouss-motherboard:MPCIE-Socket U4
+L pimouss-motherboard:MPCIE-Socket P3
 U 1 1 5E649649
 P 5450 3750
-AR Path="/5C91A44F/5D489567/5E649649" Ref="U4"  Part="1"
-AR Path="/5C91A44F/5D9F9D59/5E649649" Ref="U5"  Part="1"
-F 0 "U4" H 5450 5293 60  0000 C CNN
+AR Path="/5C91A44F/5D489567/5E649649" Ref="P3"  Part="1"
+AR Path="/5C91A44F/5D9F9D59/5E649649" Ref="P4"  Part="1"
+F 0 "P3" H 5450 5293 60  0000 C CNN
 F 1 "MPCIE-Socket" H 5450 5187 60  0000 C CNN
 F 2 "pimouss-motherboard:mpcie-socket" H 5450 5081 60  0000 C CNN
